File: NordiCoin.kicad_sch (KiCad schematic)
At the start: 0 parts

Commit message: added mcus
Parts:
- added M1: MDBT42T, MDBT42T, symbol NordiCoin:MDBT42T
- added M2: MDBT42TV, MDBT42TV, symbol NordiCoin:MDBT42TV
Connections:
- new net DCC: M1.17 (DCC), M2.16 (DCC)
- new net DEC4: M1.18 (DEC4), M2.17 (DEC4)
- new net GND: M1.1 (GND), M1.10 (GND), M1.16 (GND), M1.19 (GND), M2.1 (GND), M2.15 (GND), M2.19 (GND), M2.7 (GND)
- new net PO0/XL1: M1.14 (P0.00/XL1), M2.12 (P0.00/XL1)
- new net PO12: M1.9 (P0.12), M2.6 (P0.12)
- new net PO14: M1.6 (P0.14), M2.13 (P0.14)
- new net PO16: M1.8 (P0.16), M2.11 (P0.16)
- new net PO18: M1.7 (P0.18), M2.5 (P0.18)
- new net PO1/XL2: M1.13 (P0.01/XL2), M2.10 (P0.01/XL2)
- new net PO20: M1.5 (P0.20), M2.18 (P0.20)
- new net PO21/RESET: M1.4 (P0.21/RESET), M2.4 (P0.21/RESET)
- new net PO4: M1.12 (P0.04), M2.8 (P0.04)
- new net PO5: M1.11 (P0.05), M2.9 (P0.05)
- new net SWDCLK: M1.3 (SWDCLK), M2.3 (SWDCLK)
- new net SWDIO: M1.2 (SWDIO), M2.2 (SWDIO)
- new net VCC: M1.15 (VDD), M2.14 (VDD)

Commit message: Layout done
Parts:
- added BT1: Battery_Cell, NordiCoin:BAT_120591-1, symbol Device:Battery_Cell
- added BZ1: Buzzer, NordiCoin:AST0760_MAL, symbol Device:Buzzer
- added C1, C5: 100n, Capacitor_SMD:C_0603_1608Metric, symbol Device:C
- added C2: 1u, Capacitor_SMD:C_0603_1608Metric, symbol Device:C
- added C3, C4: 12p, Capacitor_SMD:C_0402_1005Metric, symbol Device:C
- added D2: LED, LED_SMD:LED_0603_1608Metric, symbol Device:LED
- added J1: Conn_01x05_Pin, Connector_PinHeader_1.00mm:PinHeader_1x05_P1.00mm_Vertical, symbol Connector:Conn_01x05_Pin
- added JP1, JP2, JP3: Jumper_2_Small_Open, NordiCoin:SolderJumper_UnBridged_Small, symbol Jumper:Jumper_2_Small_Open
- added Q4: FDN304PZ, Package_TO_SOT_SMD:SOT-23, symbol Watchy:BSS83P
- added R1, R3, R4: 1K, Capacitor_SMD:C_0402_1005Metric, symbol Device:R
- added R2: 100K, Capacitor_SMD:C_0402_1005Metric, symbol Device:R
- added SW1: SW_Push, NordiCoin:SW4_PTS815 SJM 250 SMTR LFS_CNK, symbol Switch:SW_Push
- added Y1: ABS07-32.768KHZ-T, NordiCoin:XTAL_9HT10_TXC, symbol Device:Crystal
- M1: footprint MDBT42T -> NordiCoin:MDBT42T
- M2: footprint MDBT42TV -> NordiCoin:MDBT42TV
Connections:
- net GND: now also BT1.2 (-), BZ1.2 (-), C1.2, C2.2, C3.2, C4.2, C5.2, J1.5 (Pin_5), R2.1, R4.1
- net PO0/XL1: now also C4.1, JP3.1 (A), Y1.2; no longer M2.12 (P0.00/XL1)
- net PO16: now also R4.2, SW1.1
- net PO18: now also R3.1
- net PO1/XL2: now also C3.1, JP1.1 (A), Y1.1; no longer M2.10 (P0.01/XL2)
- net PO20: now also D2.1 (K)
- net PO21/RESET: now also J1.4 (Pin_4)
- net SWDCLK: now also J1.2 (Pin_2)
- net SWDIO: now also J1.3 (Pin_3)
- net VCC: now also C1.1, C2.1, J1.1 (Pin_1), JP2.2 (B), Q4.2 (S), R1.2, SW1.2
- new net: C5.1, Q4.1 (G), R2.2
- new net: D2.2 (A), R1.1
- new net: JP1.2 (B), M2.10 (P0.01/XL2)
- new net: JP3.2 (B), M2.12 (P0.00/XL1)
- new net: BZ1.1 (+), R3.2
- new net +BATT: BT1.1 (+), JP2.1 (A), Q4.3 (D)
Other:
- note added: "Batt is too far away"
- note added: "Optional"
