File: NordiCoin.kicad_pcb (KiCad board)
At the start: 2 copper layers, 20.5 x 29.8 mm, 21 parts, among them J1 Conn_01x05_Pin, M1 MDBT42T, M2 MDBT42TV, Q4 FDN304PZ, SW1 SW_Push, Y1 ABS07-32.768KHZ-T

Commit message: done maybe
Routing:
- net GND: track 0.00 -> 97.4 mm, vias 0 -> 41
- net VCC: track 0.00 -> 39.8 mm, vias 0 -> 4
- net PO16: track 0.00 -> 39.8 mm, vias 0 -> 3
- net PO14: track 0.00 -> 28.6 mm, vias 0 -> 2
- net PO18: track 0.00 -> 28.3 mm, vias 0 -> 4
- net SWDCLK: track 0.00 -> 24.6 mm, vias 0 -> 1
- net PO12: track 0.00 -> 23.4 mm, vias 0 -> 4
- net SWDIO: track 0.00 -> 21.3 mm, vias 0 -> 1
- net PO21/RESET: track 0.00 -> 20.9 mm, vias 0 -> 2
- net DEC4: track 0.00 -> 16.8 mm, vias 0 -> 2
- net DCC: track 0.00 -> 16.2 mm, vias 0 -> 2
- net PO5: track 0.00 -> 15.3 mm, vias 0 -> 2
- net PO4: track 0.00 -> 13.7 mm
- net PO0/XL1: track 0.00 -> 11.9 mm, vias 0 -> 2
- net PO1/XL2: track 0.00 -> 11.6 mm, vias 0 -> 2
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Other:
- board text added: "NordiCoin"
- board text added: "by Szybet"

Commit message: done
Parts:
- moved R1 0.14 mm to (129.3, 68.3)
Routing:
- net GND: vias 41 -> 40
