File: hardware/NordiCoin.kicad_pcb (KiCad board)
At the start: 2 copper layers, 20.5 x 29.8 mm, 21 parts, among them J1 Conn_01x05_Pin, M1 MDBT42T, M2 MDBT42TV, Q4 FDN304PZ, SW1 SW_Push, Y1 ABS07-32.768KHZ-T

Commit message: some pcb adjustments
Parts:
- removed R4: 1K, Capacitor_SMD:C_0402_1005Metric
- R1, R3: value 1K -> 330R
Routing:
- net GND: track 97.4 -> 89.8 mm
- net PO16: track 39.8 -> 38.3 mm
